File: hardware/sensors-and-control/sensors-and-control.sch (EAGLE design)
At the start: 132 parts, among them IC1 STM32L496ZET6

Commit message: fixed flush button to use unused EXTI pin
Parts:
- removed U$30: NC, voltage-ground:NC
- added U$14, U$29: NC, voltage-ground:NC
Connections:
- net LM_ENC_OUT_A renamed LM_ENC_A
- net LM_ENC_OUT_B renamed LM_ENC_B
- net LM_PWM_IN1 renamed LM_PWM_1
- net LM_PWM_IN2 renamed LM_PWM_2
- net RM_ENC_OUT_A renamed RM_ENC_A
- net RM_ENC_OUT_B renamed RM_ENC_B
- net RM_PWM_IN1 renamed RM_PWM_1
- net RM_PWM_IN2 renamed RM_PWM_2
- removed net N$46: IC1_A.104-PA12, U$30.1
- new net N$30: IC1_A.103-PA11, U$14.1
- new net N$45: IC1_G.132-PG15, U$29.1
- net SD_FLUSH: now also IC1_A.104-PA12; no longer IC1_A.103-PA11
Changed lines of the file:
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@@
 <part name="U$27" library="voltage-ground" library_urn="urn:adsk.eagle:library:704746" deviceset="NC" device=""/>
 <part name="U$28" library="voltage-ground" library_urn="urn:adsk.eagle:library:704746" deviceset="NC" device=""/>
-<part name="U$30" library="voltage-ground" library_urn="urn:adsk.eagle:library:704746" deviceset="NC" device=""/>
 <part name="U$31" library="voltage-ground" library_urn="urn:adsk.eagle:library:704746" deviceset="NC" device=""/>
 <part name="U$32" library="voltage-ground" library_urn="urn:adsk.eagle:library:704746" deviceset="NC" device=""/>
@@
 <part name="DGND56" library="voltage-ground" library_urn="urn:adsk.eagle:library:704746" deviceset="DGND" device=""/>
 <part name="R27" library="resistors" library_urn="urn:adsk.eagle:library:704770" deviceset="RESISTOR_0.1W" device="" package3d_urn="urn:adsk.eagle:package:704947/3" value="15k"/>
+<part name="U$14" library="voltage-ground" library_urn="urn:adsk.eagle:library:704746" deviceset="NC" device=""/>
+<part name="U$29" library="voltage-ground" library_urn="urn:adsk.eagle:library:704746" deviceset="NC" device=""/>
 </parts>
 <sheets>
@@
 <instance part="U$27" gate="G$1" x="73.66" y="73.66" rot="R180"/>
 <instance part="U$28" gate="G$1" x="73.66" y="38.1" rot="R180"/>
-<instance part="U$30" gate="G$1" x="73.66" y="27.94" rot="R180"/>
 <instance part="U$31" gate="G$1" x="33.02" y="38.1"/>
 <instance part="U$32" gate="G$1" x="33.02" y="40.64"/>
@@
 <instance part="U$35" gate="G$1" x="33.02" y="30.48"/>
 <instance part="U$36" gate="G$1" x="33.02" y="22.86"/>
+<instance part="U$14" gate="G$1" x="73.66" y="30.48" rot="R180"/>
+<instance part="U$29" gate="G$1" x="129.54" y="165.1"/>
 </instances>
 <busses>
@@
 </segment>
 </net>
-<net name="RM_ENC_OUT_A" class="0">
+<net name="RM_ENC_A" class="0">
 <segment>
 <pinref part="IC1" gate="_D" pin="81-PD12"/>
@@
 </segment>
 </net>
-<net name="RM_ENC_OUT_B" class="0">
+<net name="RM_ENC_B" class="0">
 <segment>
 <pinref part="IC1" gate="_B" pin="75-PB14"/>
@@
 </segment>
 </net>
-<net name="RM_PWM_IN1" class="0">
+<net name="RM_PWM_1" class="0">
 <segment>
 <pinref part="IC1" gate="_B" pin="48-PB2"/>
@@
 </segment>
 </net>
-<net name="RM_PWM_IN2" class="0">
+<net name="RM_PWM_2" class="0">
 <segment>
 <pinref part="IC1" gate="_D" pin="82-PD13"/>
@@
 </segment>
 </net>
-<net name="N$46" class="0">
-<segment>
-<pinref part="IC1" gate="_A" pin="104-PA12"/>
-<pinref part="U$30" gate="G$1" pin="1"/>
-</segment>
-</net>
 <net name="N$47" class="0">
 <segment>
@@
 <pinref part="IC1" gate="_B" pin="47-PB1"/>
 <pinref part="U$36" gate="G$1" pin="1"/>
-</segment>
-</net>
-<net name="SD_FLUSH" class="0">
-<segment>
-<pinref part="IC1" gate="_A" pin="103-PA11"/>
-<wire x1="76.2" y1="30.48" x2="55.88" y2="30.48" width="0.1524" layer="91"/>
-<label x="58.42" y="30.48" size="1.778" layer="95"/>
 </segment>
 </net>
@@
 <wire x1="127" y1="83.82" x2="152.4" y2="83.82" width="0.1524" layer="91"/>
 <label x="129.54" y="83.82" size="1.778" layer="95"/>
+</segment>
+</net>
+<net name="SD_FLUSH" class="0">
+<segment>
+<pinref part="IC1" gate="_A" pin="104-PA12"/>
+<wire x1="76.2" y1="27.94" x2="55.88" y2="27.94" width="0.1524" layer="91"/>
+<label x="58.42" y="27.94" size="1.778" layer="95"/>
+</segment>
+</net>
+<net name="N$30" class="0">
+<segment>
+<pinref part="IC1" gate="_A" pin="103-PA11"/>
+<pinref part="U$14" gate="G$1" pin="1"/>
+</segment>
+</net>
+<net name="N$45" class="0">
+<segment>
+<pinref part="IC1" gate="_G" pin="132-PG15"/>
+<pinref part="U$29" gate="G$1" pin="1"/>
 </segment>
 </net>
@@
 </segment>
 </net>
-<net name="RM_ENC_OUT_B" class="0">
+<net name="RM_ENC_B" class="0">
 <segment>
 <pinref part="RIGHT_MOTOR_ENCODER" gate="G$1" pin="2"/>
@@
 </segment>
 </net>
-<net name="RM_ENC_OUT_A" class="0">
+<net name="RM_ENC_A" class="0">
 <segment>
 <pinref part="RIGHT_MOTOR_ENCODER" gate="G$1" pin="3"/>
@@
 </segment>
 </net>
-<net name="LM_ENC_OUT_A" class="0">
+<net name="LM_ENC_A" class="0">
 <segment>
 <pinref part="LEFT_MOTOR_ENCODER" gate="G$1" pin="3"/>
@@
 </segment>
 </net>
-<net name="LM_ENC_OUT_B" class="0">
+<net name="LM_ENC_B" class="0">
 <segment>
 <pinref part="LEFT_MOTOR_ENCODER" gate="G$1" pin="2"/>
@@
 </segment>
 </net>
-<net name="LM_PWM_IN1" class="0">
+<net name="LM_PWM_1" class="0">
 <segment>
 <pinref part="IC1" gate="_E" pin="141-PE0"/>
@@
 </segment>
 </net>
-<net name="LM_PWM_IN2" class="0">
+<net name="LM_PWM_2" class="0">
 <segment>
 <pinref part="IC1" gate="_E" pin="142-PE1"/>
@@
 </segment>
 </net>
-<net name="RM_PWM_IN2" class="0">
+<net name="RM_PWM_2" class="0">
 <segment>
 <pinref part="RIGHT_MOTOR_CONTROL" gate="G$1" pin="3"/>
@@
 </segment>
 </net>
-<net name="RM_PWM_IN1" class="0">
+<net name="RM_PWM_1" class="0">
 <segment>
 <pinref part="RIGHT_MOTOR_CONTROL" gate="G$1" pin="4"/>
