File: hardware/line-sensor/line-sensor-r2.sch (EAGLE design)
At the start: 97 parts, among them IC1 GP2S60, IC10 GP2S60, IC11 GP2S60, IC12 GP2S60, IC13 GP2S60, IC14 GP2S60, IC15 GP2S60, IC16 GP2S60, IC17 GP2S60, IC18 GP2S60, IC19 GP2S60, IC2 GP2S60, IC20 GP2S60, IC21 GP2S60, IC22 GP2S60, IC23 GP2S60, IC3 GP2S60, IC4 GP2S60, IC5 GP2S60, IC6 GP2S60, IC7 GP2S60, IC8 GP2S60, IC9 GP2S60

Commit message: - added voltage sources for line sensor (not complete)
Parts:
- removed JP1: MOLEX-501931-3070, connectors:MOLEX-501931-3070
- added C10, C13, C14, C15, C16, C17, C18: 0.1u, capacitors:CAPACITOR0603
- added C11: 33n 10V X7R, capacitors:CAPACITOR0603
- added C12: 4.7u, capacitors:CAPACITOR0805
- added C19: 22u 10V X7R, capacitors:CAPACITOR0805
- added C3, C4: 1u 10V X7R, capacitors:CAPACITOR0805
- added C5: 1u, capacitors:CAPACITOR0603
- added C6: 1u 50V X7R, capacitors:CAPACITOR1206
- added C7: 22u 10V X7S, capacitors:CAPACITOR0805
- added C8: 0.1u 10V X7R, capacitors:CAPACITOR0603
- added C9: 10u 50V X7R, capacitors:CAPACITOR0805
- added IC24: STM32L151VE, mcu:STM32L151VE
- added IC25, IC26: GP2S60, sensors:GP2S60
- added IC27: ADR366BUJZ, voltage-source:ADR366BUJZ
- added IC28: TI-TPS62170, voltage-source:TI-TPS62170
- added IC29: TI-LM5165YDRCR, voltage-source:TI-LM5165YDRCR
- added IC30: ADP124ARHZ-3.3-R7CT-ND, voltage-source:ADP124ARHZ-3.3-R7CT-ND
- added L1: 3.3u 2.63A, inductors:VLS3012HBX
- added L2: 150u 0.35A, inductors:ELL-6SH151M
- added R47, R49: 1k, resistors:RESISTOR_0.1W
- added R48, R50: 220k, resistors:RESISTOR_0.1W
- added R51: 121k 1%, resistors:RESISTOR_0.1W
- added R52: 100k 1%, resistors:RESISTOR_0.1W
- added R53: 0.5 1%, resistors:RESISTOR_0.1W
- added R54: 100k, resistors:RESISTOR_0.1W
- added R55: 610k 1%, resistors:RESISTOR_0.1W
- added R56: 180k 1%, resistors:RESISTOR_0.1W
- added SUPPLY26, SUPPLY27, SUPPLY28: +VBAT, voltage-ground:+VBAT
- added SUPPLY29, SUPPLY30, SUPPLY31, SUPPLY32, SUPPLY33, SUPPLY34: +3.3V, voltage-ground:+3.3V
- added U$1, U$2, U$3, U$4, U$5, U$6: NC, voltage-ground:NC
- C1: value 0.1u -> 0.1u 10V
- C2: value 10u -> 0.1u 50V
Connections:
- new net !RST: C18.1, IC24PWR&AUX.!RST!
- new net 3V1: R47.2, R48.2, SUPPLY2.VCC
- new net 3V2: R49.2, R50.2, SUPPLY25.VCC
- new net BOOT0: IC24PWR&AUX.BOOT0, R54.1
- new net DGND: C10.2, C11.2, C12.2, C13.2, C14.2, C15.2, C16.2, C17.2, C18.2, C7.2, IC24PWR&AUX.VSS_1, IC24PWR&AUX.VSS_2, IC24PWR&AUX.VSS_3, IC24PWR&AUX.VSS_4, IC24PWR&AUX.VSS_5, IC29.GND, IC29.ILIM, IC29.PAD, R54.2
- new net GND: C19.2, C2.2, C4.2, C6.2, C9.2, IC27.GND, IC28.AGND, IC28.PAD, IC28.PGND, R51.2, R56.1
- new net N$24: IC25.4, R47.1
- new net N$25: IC26.4, R49.1
- new net N$26: IC28.SW, L1.P$1
- new net N$27: IC28.PG, R52.1
- new net N$28: C11.1, IC29.SS
- new net N$29: IC29.SW, L2.P$1
- new net N$30: IC29.RT, R51.1
- new net N$31: IC28.FB, R55.1, R56.2
- new net N$32: C7.1, R53.2
- new net SENSOR_24: IC24B.PB14, IC25.1, R48.1
- new net SENSOR_25: IC24B.PB15, IC26.1, R50.1
- new net V3.5: C19.1, C4.1, IC28.VOS, IC30.EN, IC30.VIN_1, IC30.VIN_2, L1.P$2, R52.2, R55.2
- new net VBAT: C2.1, C6.1, C9.1, IC27.VIN, IC28.EN, IC28.VIN, IC29.EN, IC29.VIN, SUPPLY26.VCC, SUPPLY27.VCC, SUPPLY28.VCC
- new net VDD: C10.1, C12.1, C13.1, C14.1, C15.1, C16.1, C17.1, IC24PWR&AUX.VDD_1, IC24PWR&AUX.VDD_2, IC24PWR&AUX.VDD_3, IC24PWR&AUX.VDD_4, IC24PWR&AUX.VDD_5, IC24PWR&AUX.VLCD, IC29.VOUT, L2.P$2, R53.1, SUPPLY29.VCC, SUPPLY30.VCC, SUPPLY31.VCC, SUPPLY32.VCC, SUPPLY33.VCC, SUPPLY34.VCC
- new net VDDA: C3.1, C8.1, IC24PWR&AUX.VDDA, IC30.VOUT_1, IC30.VOUT_2, IC30.VOUT_SENSE
- new net VREF3.3: C1.1, C5.1, IC24PWR&AUX.VREF+, IC27.VOUT
- net 3V3: no longer C1.1, C2.1, JP1.1, JP1.3, JP1.30, SUPPLY2.VCC, SUPPLY25.VCC
- net AGND: now also C3.2, C5.2, C8.2, IC24PWR&AUX.VREF-, IC24PWR&AUX.VSSA, IC25.2, IC25.3, IC26.2, IC26.3, IC30.GND; no longer C2.2, JP1.2, JP1.28, JP1.29, JP1.4, JP1.N1, JP1.N2, JP1.N3, JP1.N4
- net SENSOR_1: now also IC24C.PC0; no longer JP1.5
- net SENSOR_10: now also IC24A.PA5; no longer JP1.14
- net SENSOR_11: now also IC24A.PA6; no longer JP1.15
- net SENSOR_12: now also IC24A.PA7; no longer JP1.16
- net SENSOR_13: now also IC24C.PC4; no longer JP1.17
- net SENSOR_14: now also IC24C.PC5; no longer JP1.18
- net SENSOR_15: now also IC24B.PB0; no longer JP1.19
- net SENSOR_16: now also IC24B.PB1; no longer JP1.20
- net SENSOR_17: now also IC24B.PB2; no longer JP1.21
- net SENSOR_18: now also IC24E.PE7; no longer JP1.22
- net SENSOR_19: now also IC24E.PE8; no longer JP1.23
- net SENSOR_2: now also IC24C.PC1; no longer JP1.6
- net SENSOR_20: now also IC24E.PE9; no longer JP1.24
- net SENSOR_21: now also IC24E.PE10; no longer JP1.25
- net SENSOR_22: now also IC24B.PB12; no longer JP1.26
- net SENSOR_23: now also IC24B.PB13; no longer JP1.27
- net SENSOR_3: now also IC24C.PC2; no longer JP1.7
- net SENSOR_4: now also IC24C.PC3; no longer JP1.8
- net SENSOR_5: now also IC24A.PA0/WKUP1; no longer JP1.9
- net SENSOR_6: now also IC24A.PA1; no longer JP1.10
- net SENSOR_7: now also IC24A.PA2; no longer JP1.11
- net SENSOR_8: now also IC24A.PA3; no longer JP1.12
- net SENSOR_9: now also IC24A.PA4; no longer JP1.13
Other:
- note added: "ADC and sensors power supply"
- note added: "MCU"
- note added: "MCU power supply"
- note added: "Power"
- note added: "Reference voltage for ADC"
- note added: "Sensors 1/2"
- note added: "Sensors 2/2"
- note added: "add voltage calculation and check effect of tolerance +/- 1% on output voltage"
- note added: "wrong part (current one has current 5ma but chip needs 7ma) switch to ADR3533WBRMZ-R7 need to also check max V i need after I test sensors with a bunch of resistors on lines and all black"
- note removed: "Sensors"
- note removed: "Sensors Power"

Commit message: - added line sensor power layout and mcu pin usage configuration
Parts:
- removed U$1, U$2, U$3, U$4, U$5, U$6: NC, voltage-ground:NC
- added C20: 0.1u 10V X7R, capacitors:CAPACITOR0603
- added J1: MOLEX-502382-02XX, connectors:MOLEX-502382-02XX
- added J2: MOLEX-502382-05XX, connectors:MOLEX-502382-05XX
- added J3: MOLEX-53261-0771, connectors:MOLEX-53261-0771
- added R57, R58, R59, R60, R61, R62, R63, R64, R65: 0, resistors:RESISTOR_0.1W
- C1: value 0.1u 10V -> 0.1u
- C10: value 0.1u -> 33n 10V X7R
- C11: value 33n 10V X7R -> 22u 10V X7S; device capacitors:CAPACITOR0603 -> capacitors:CAPACITOR0805
- C13: value 0.1u -> 22u 10V X7R; device capacitors:CAPACITOR0603 -> capacitors:CAPACITOR0805
- C14: value 0.1u -> 10u 50V
- C15, C18: value 0.1u -> 1u 10V X7R; device capacitors:CAPACITOR0603 -> capacitors:CAPACITOR0805
- C16: value 0.1u -> 0.1u 50V
- C17: value 0.1u -> 1u 10V Tant; device capacitors:CAPACITOR0603 -> capacitors:CAPACITOR_POLARIZED
- C19: value 22u 10V X7R -> 0.1u 10V X7R; device capacitors:CAPACITOR0805 -> capacitors:CAPACITOR0603
- C2: value 0.1u 50V -> 0.1u
- C3, C4: value 1u 10V X7R -> 0.1u; device capacitors:CAPACITOR0805 -> capacitors:CAPACITOR0603
- C5: value 1u -> 0.1u
- C6: value 1u 50V X7R -> 0.1u; device capacitors:CAPACITOR1206 -> capacitors:CAPACITOR0603
- C7: value 22u 10V X7S -> 0.1u; device capacitors:CAPACITOR0805 -> capacitors:CAPACITOR0603
- C8: value 0.1u 10V X7R -> 10u 50V X7R; device capacitors:CAPACITOR0603 -> capacitors:CAPACITOR0805
- C9: value 10u 50V X7R -> 1u 50V X7R; device capacitors:CAPACITOR0805 -> capacitors:CAPACITOR1206
- IC24: value STM32L151VE -> GP2S60; device mcu:STM32L151VE -> sensors:GP2S60
- IC26: value GP2S60 -> STM32L151VE; device sensors:GP2S60 -> mcu:STM32L151VE
- IC27: value ADR366BUJZ -> TI-LM5165YDRCR; device voltage-source:ADR366BUJZ -> voltage-source:TI-LM5165YDRCR
- IC29: value TI-LM5165YDRCR -> AD-REF196GSZ; device voltage-source:TI-LM5165YDRCR -> voltage-source:AD-REF196GSZ
- IC30: value ADP124ARHZ-3.3-R7CT-ND -> AD-ADP124ARHZ; device voltage-source:ADP124ARHZ-3.3-R7CT-ND -> voltage-source:AD-ADP124ARHZ
- R10, R14, R18, R2, R22, R26, R30, R34, R38, R42, R6: value 220k -> 1k
- R11, R15, R19, R23, R27, R3, R31, R35, R39, R43, R7: value 1k -> 220k
- R51: value 121k 1% -> 100k
- R52: value 100k 1% -> 121k 1%
- R53: value 0.5 1% -> 100k 1%
- R54: value 100k -> 0.5 1%
- SUPPLY26, SUPPLY27, SUPPLY28: value +VBAT -> +3.3V; device voltage-ground:+VBAT -> voltage-ground:+3.3V
- SUPPLY32, SUPPLY33, SUPPLY34: value +3.3V -> +VBAT; device voltage-ground:+3.3V -> voltage-ground:+VBAT
Connections:
- net N$26 renamed IC28_SW
- removed net AGND: C1.2, C3.2, C5.2, C8.2, IC1.2, IC1.3, IC10.2, IC10.3, IC11.2, IC11.3, IC12.2, IC12.3, IC13.2, IC13.3, IC14.2, IC14.3, IC15.2, IC15.3, IC16.2, IC16.3, IC17.2, IC17.3, IC18.2, IC18.3, IC19.2, IC19.3, IC2.2, IC2.3, IC20.2, IC20.3, IC21.2, IC21.3, IC22.2, IC22.3, IC23.2, IC23.3, IC24PWR&AUX.VREF-, IC24PWR&AUX.VSSA, IC25.2, IC25.3, IC26.2, IC26.3, IC3.2, IC3.3, IC30.GND, IC4.2, IC4.3, IC5.2, IC5.3, IC6.2, IC6.3, IC7.2, IC7.3, IC8.2, IC8.3, IC9.2, IC9.3
- removed net DGND: C10.2, C11.2, C12.2, C13.2, C14.2, C15.2, C16.2, C17.2, C18.2, C7.2, IC24PWR&AUX.VSS_1, IC24PWR&AUX.VSS_2, IC24PWR&AUX.VSS_3, IC24PWR&AUX.VSS_4, IC24PWR&AUX.VSS_5, IC29.GND, IC29.ILIM, IC29.PAD, R54.2
- removed net N$1 (its old number): IC2.4, R3.1
- removed net N$16 (its old number): IC16.4, R31.1
- removed net N$18 (its old number): IC18.4, R35.1
- removed net N$30: IC29.RT, R51.1
- removed net N$32: C7.1, R53.2
- removed net N$4 (its old number): IC4.4, R7.1
- removed net N$6 (its old number): IC6.4, R11.1
- removed net V3.5: C19.1, C4.1, IC28.VOS, IC30.EN, IC30.VIN_1, IC30.VIN_2, L1.P$2, R52.2, R55.2
- new net I2C1_SCL: IC26B.PB6, R60.1
- new net I2C1_SDA: IC26B.PB7, R57.1
- new net I2C1_SMBA: IC26B.PB5, R64.2
- new net IC27_SW: IC27.SW, L2.P$1
- new net N$11: IC10.4, R18.1
- new net N$13: IC12.4, R22.1
- new net N$21: IC25.4, R49.1
- new net N$23: IC18.4, R34.1
- new net N$26: J2.2, R57.2, R58.2, R59.2
- new net N$33: IC27.RT, R52.1
- new net N$34: C10.1, IC27.SS
- new net N$36: C11.1, R54.2
- new net N$38: IC28.PG, R53.1
- new net N$9: IC6.4, R10.1
- new net SPI3_MISO: IC26C.PC11, R62.1
- new net SPI3_MOSI: IC26C.PC12, R59.1
- new net SPI3_NSS: IC26A.PA15, R65.2
- new net SPI3_SCK: IC26C.PC10, R63.2
- new net STLINK_SWO: IC26B.PB3, J3.5
- new net STLINK_TCK: IC26A.PA14, J3.6
- new net STLINK_TMS: IC26A.PA13, J3.4
- new net STLINK_USART1_RX: IC26A.PA10, J3.3
- new net STLINK_USART1_TX: IC26A.PA9, J3.2
- new net USART2_RX: IC26D.PD6, R58.1
- new net USART2_TX: IC26D.PD5, R61.1
- new net VDDA3.5: C13.1, C15.1, IC28.VOS, IC30.EN, IC30.VIN_1, IC30.VIN_2, L1.P$2, R53.2, R55.2
- net !RST: now also C6.1, IC26PWR&AUX.!RST!, J3.1; no longer C18.1, IC24PWR&AUX.!RST!
- net 3V1: now also R38.2, R40.2, SUPPLY20.VCC; no longer R47.2, R48.2, SUPPLY2.VCC
- net 3V2: now also R42.2, R44.2, SUPPLY22.VCC; no longer R49.2, R50.2, SUPPLY25.VCC
- net 3V3: now also R47.2, R48.2, R49.2, R50.2, SUPPLY2.VCC, SUPPLY25.VCC; no longer R38.2, R40.2, R42.2, R44.2, SUPPLY20.VCC, SUPPLY22.VCC
- net BOOT0: now also IC26PWR&AUX.BOOT0, R51.1; no longer IC24PWR&AUX.BOOT0, R54.1
- net GND: now also C1.2, C10.2, C11.2, C12.2, C13.2, C14.2, C15.2, C16.2, C17.NEG, C18.2, C20.2, C3.2, C5.2, C7.2, C8.2, IC1.2, IC1.3, IC10.2, IC10.3, IC11.2, IC11.3, IC12.2, IC12.3, IC13.2, IC13.3, IC14.2, IC14.3, IC15.2, IC15.3, IC16.2, IC16.3, IC17.2, IC17.3, IC18.2, IC18.3, IC19.2, IC19.3, IC2.2, IC2.3, IC20.2, IC20.3, IC21.2, IC21.3, IC22.2, IC22.3, IC23.2, IC23.3, IC24.2, IC24.3, IC25.2, IC25.3, IC26PWR&AUX.VREF-, IC26PWR&AUX.VSSA, IC26PWR&AUX.VSS_1, IC26PWR&AUX.VSS_2, IC26PWR&AUX.VSS_3, IC26PWR&AUX.VSS_4, IC26PWR&AUX.VSS_5, IC27.ILIM, IC27.PAD, IC29.GND, IC3.2, IC3.3, IC30.GND, IC30.PAD, IC4.2, IC4.3, IC5.2, IC5.3, IC6.2, IC6.3, IC7.2, IC7.3, IC8.2, IC8.3, IC9.2, IC9.3, J1.2, J1.G1, J1.G2, J2.1, J2.G1, J2.G2, J3.7, J3.G1, J3.G2, R52.2
- net N$10: now also IC8.4, R14.1; no longer IC10.4, R19.1
- net N$12: now also IC2.4, R2.1; no longer IC12.4, R23.1
- net N$14: now also R26.1; no longer R27.1
- net N$20: now also IC24.4, R47.1; no longer IC20.4, R39.1
- net N$22: now also IC16.4, R30.1; no longer IC22.4, R43.1
- net N$24: now also IC20.4, R38.1; no longer IC25.4, R47.1
- net N$25: now also IC22.4, R42.1; no longer IC26.4, R49.1
- net N$27: now also J2.3, R60.2, R61.2, R62.2; no longer IC28.PG, R52.1
- net N$28: now also J2.4, R63.1, R64.1; no longer C11.1, IC29.SS
- net N$29: now also J2.5, R65.1; no longer IC29.SW, L2.P$1
- net N$8: now also IC4.4, R6.1; no longer IC8.4, R15.1
- net SENSOR_1: now also IC26C.PC0, R3.1; no longer IC24C.PC0, R2.1
- net SENSOR_10: now also IC26A.PA5, IC8.1, R16.1; no longer IC10.1, IC24A.PA5, R20.1
- net SENSOR_11: now also IC10.1, IC26A.PA6, R20.1; no longer IC11.1, IC24A.PA6, R22.1
- net SENSOR_12: now also IC2.1, IC26A.PA7, R4.1; no longer IC12.1, IC24A.PA7, R24.1
- net SENSOR_13: now also IC12.1, IC26C.PC4, R24.1; no longer IC13.1, IC24C.PC4, R26.1
- net SENSOR_14: now also IC26C.PC5; no longer IC24C.PC5
- net SENSOR_15: now also IC26B.PB0, R31.1; no longer IC24B.PB0, R30.1
- net SENSOR_16: now also IC17.1, IC26B.PB1, R35.1; no longer IC16.1, IC24B.PB1, R32.1
- net SENSOR_17: now also IC19.1, IC26B.PB2, R39.1; no longer IC17.1, IC24B.PB2, R34.1
- net SENSOR_18: now also IC21.1, IC26E.PE7, R43.1; no longer IC18.1, IC24E.PE7, R36.1
- net SENSOR_19: now also IC23.1, IC26E.PE8, R46.1; no longer IC19.1, IC24E.PE8, R38.1
- net SENSOR_2: now also IC26C.PC1, IC3.1, R7.1; no longer IC2.1, IC24C.PC1, R4.1
- net SENSOR_20: now also IC24.1, IC26E.PE9, R48.1; no longer IC20.1, IC24E.PE9, R40.1
- net SENSOR_21: now also IC25.1, IC26E.PE10, R50.1; no longer IC21.1, IC24E.PE10, R42.1
- net SENSOR_22: now also IC16.1, IC26B.PB12, R32.1; no longer IC22.1, IC24B.PB12, R44.1
- net SENSOR_23: now also IC18.1, IC26B.PB13, R36.1; no longer IC23.1, IC24B.PB13, R46.1
- net SENSOR_24: now also IC20.1, IC26B.PB14, R40.1; no longer IC24B.PB14, IC25.1, R48.1
- net SENSOR_25: now also IC22.1, IC26B.PB15, R44.1; no longer IC24B.PB15, IC26.1, R50.1
- net SENSOR_3: now also IC26C.PC2, IC5.1, R11.1; no longer IC24C.PC2, IC3.1, R6.1
- net SENSOR_4: now also IC26C.PC3, IC7.1, R15.1; no longer IC24C.PC3, IC4.1, R8.1
- net SENSOR_5: now also IC26A.PA0/WKUP1, IC9.1, R19.1; no longer IC24A.PA0/WKUP1, IC5.1, R10.1
- net SENSOR_6: now also IC11.1, IC26A.PA1, R23.1; no longer IC24A.PA1, IC6.1, R12.1
- net SENSOR_7: now also IC13.1, IC26A.PA2, R27.1; no longer IC24A.PA2, IC7.1, R14.1
- net SENSOR_8: now also IC26A.PA3, IC4.1, R8.1; no longer IC24A.PA3, IC8.1, R16.1
- net SENSOR_9: now also IC26A.PA4, IC6.1, R12.1; no longer IC24A.PA4, IC9.1, R18.1
- net VBAT: now also C14.1, C16.1, C8.1, IC27.EN, IC29.!SLEEP, IC29.VS, J1.1, SUPPLY32.VCC, SUPPLY33.VCC, SUPPLY34.VCC; no longer C2.1, C6.1, IC29.EN, IC29.VIN, SUPPLY26.VCC, SUPPLY27.VCC, SUPPLY28.VCC
- net VDD: now also C1.1, C2.1, C3.1, C4.1, C5.1, C7.1, IC26PWR&AUX.VDD_1, IC26PWR&AUX.VDD_2, IC26PWR&AUX.VDD_3, IC26PWR&AUX.VDD_4, IC26PWR&AUX.VDD_5, IC26PWR&AUX.VLCD, IC27.VOUT, R54.1, SUPPLY26.VCC, SUPPLY27.VCC, SUPPLY28.VCC; no longer C10.1, C13.1, C14.1, C15.1, C16.1, C17.1, IC24PWR&AUX.VDD_1, IC24PWR&AUX.VDD_2, IC24PWR&AUX.VDD_3, IC24PWR&AUX.VDD_4, IC24PWR&AUX.VDD_5, IC24PWR&AUX.VLCD, IC29.VOUT, R53.1, SUPPLY32.VCC, SUPPLY33.VCC, SUPPLY34.VCC
- net VDDA: now also C18.1, C20.1, IC26PWR&AUX.VDDA; no longer C3.1, C8.1, IC24PWR&AUX.VDDA
- net VREF3.3: now also C17.POS, C19.1, IC26PWR&AUX.VREF+, IC29.OUT; no longer C1.1, C5.1, IC24PWR&AUX.VREF+, IC27.VOUT
Other:
- note added: "ADC power supply ADC reference voltage Sensors power supply"
- note added: "Battery"
- note added: "R4/R5 are used to set output voltage R5 must be < 400k VDDA3.5 voltage range: min = 3.45743 (smaller R4, larger R5) max = 3.56588 (larger R4, smaller R5)"
- note added: "VBAT range: min = 4V max = 14V"
- note removed: "ADC and sensors power supply"
- note removed: "Reference voltage for ADC"
- note removed: "add voltage calculation and check effect of tolerance +/- 1% on output voltage"
- note removed: "wrong part (current one has current 5ma but chip needs 7ma) switch to ADR3533WBRMZ-R7 need to also check max V i need after I test sensors with a bunch of resistors on lines and all black"

Commit message: - finished line sensor with linear regulator and voltage reference
Connections:
- removed net 3V1: R38.2, R40.2, SUPPLY20.VCC
- removed net 3V2: R42.2, R44.2, SUPPLY22.VCC
- removed net 3V3: R1.2, R10.2, R11.2, R12.2, R13.2, R14.2, R15.2, R16.2, R17.2, R18.2, R19.2, R2.2, R20.2, R21.2, R22.2, R23.2, R24.2, R25.2, R26.2, R27.2, R28.2, R29.2, R3.2, R30.2, R31.2, R32.2, R33.2, R34.2, R35.2, R36.2, R37.2, R39.2, R4.2, R41.2, R43.2, R45.2, R46.2, R47.2, R48.2, R49.2, R5.2, R50.2, R6.2, R7.2, R8.2, R9.2, SUPPLY1.VCC, SUPPLY10.VCC, SUPPLY11.VCC, SUPPLY12.VCC, SUPPLY13.VCC, SUPPLY14.VCC, SUPPLY15.VCC, SUPPLY16.VCC, SUPPLY17.VCC, SUPPLY18.VCC, SUPPLY19.VCC, SUPPLY2.VCC, SUPPLY21.VCC, SUPPLY23.VCC, SUPPLY24.VCC, SUPPLY25.VCC, SUPPLY3.VCC, SUPPLY4.VCC, SUPPLY5.VCC, SUPPLY6.VCC, SUPPLY7.VCC, SUPPLY8.VCC, SUPPLY9.VCC
- net VDDA: now also R1.2, R10.2, R11.2, R12.2, R13.2, R14.2, R15.2, R16.2, R17.2, R18.2, R19.2, R2.2, R20.2, R21.2, R22.2, R23.2, R24.2, R25.2, R26.2, R27.2, R28.2, R29.2, R3.2, R30.2, R31.2, R32.2, R33.2, R34.2, R35.2, R36.2, R37.2, R38.2, R39.2, R4.2, R40.2, R41.2, R42.2, R43.2, R44.2, R45.2, R46.2, R47.2, R48.2, R49.2, R5.2, R50.2, R6.2, R7.2, R8.2, R9.2, SUPPLY1.VCC, SUPPLY10.VCC, SUPPLY11.VCC, SUPPLY12.VCC, SUPPLY13.VCC, SUPPLY14.VCC, SUPPLY15.VCC, SUPPLY16.VCC, SUPPLY17.VCC, SUPPLY18.VCC, SUPPLY19.VCC, SUPPLY2.VCC, SUPPLY20.VCC, SUPPLY21.VCC, SUPPLY22.VCC, SUPPLY23.VCC, SUPPLY24.VCC, SUPPLY25.VCC, SUPPLY3.VCC, SUPPLY4.VCC, SUPPLY5.VCC, SUPPLY6.VCC, SUPPLY7.VCC, SUPPLY8.VCC, SUPPLY9.VCC
