File: hardware/line-sensor/var1a/line-sensor-var1a-r3.brd (EAGLE design)
At the start: 112 x 60 mm, 106 parts, among them IC1 GP2S60, IC10 GP2S60, IC11 GP2S60, IC12 GP2S60, IC13 GP2S60, IC14 GP2S60, IC15 GP2S60, IC16 GP2S60, IC17 GP2S60, IC18 GP2S60, IC19 GP2S60, IC2 GP2S60, IC20 GP2S60, IC21 GP2S60, IC22 GP2S60, IC23 GP2S60, IC24 GP2S60, IC25 GP2S60, IC26 GP2S60, IC27 GP2S60, IC28 STM32L151VE, IC3 GP2S60, IC32 LM5165YDRCR, IC4 GP2S60, IC5 GP2S60, IC6 GP2S60, IC7 GP2S60, IC8 GP2S60, IC9 GP2S60, J1 MOLEX-502382-06XX, J2 MOLEX-53261-0771, J3 MOLEX-502382-02XX, Y1 CRYSTALKYOCERA-CX3225GB24000D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, Y2 CRYSTALNDK-NX3215SA

Commit message: finished 3rd revision of line sensor
Parts:
- added C12: 1u 16V X7R, passives:CAPACITOR-0603
- J3: value MOLEX-502382-02XX -> MOLEX-502382-03XX; device connectors:MOLEX-502382-02XX -> connectors:MOLEX-502382-03XX
- moved C9 1.27 mm to (69.5, 50.0), turned to 90 degrees
- moved C10 1.25 mm to (66.5, 42.5)
- moved C11 1.25 mm to (66.5, 40.0)
- moved Y2 1.06 mm to (69.0, 41.2)
- moved C8 1.03 mm to (65.8, 45.8)
- moved Y1 0.90 mm to (68.5, 46.5)
- moved J3 0.75 mm to (75.2, 16.0)
- moved R11 0.71 mm to (40.5, 63.5)
- moved R12 0.71 mm to (64.5, 63.5)
- moved R15 0.71 mm to (44.5, 63.5)
- moved R16 0.71 mm to (68.5, 63.5)
- moved R19 0.71 mm to (48.5, 63.5)
- moved R20 0.71 mm to (72.5, 63.5)
- moved R23 0.71 mm to (52.5, 63.5)
- moved R24 0.71 mm to (80.5, 63.5)
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Connections:
- new net PWR_ENABLE: C12.1, IC32.7, J3.1
- net GND: now also C12.2, J3.3; no longer J3.2
- net VBAT: now also J3.2; no longer IC32.7, J3.1
Routing:
- net VDD: track 14.1 -> 147.9 mm, vias 3 -> 38
- net SENSOR_1: track 0.00 -> 61.6 mm, vias 0 -> 3
- net SENSOR_25: track 0.00 -> 59.5 mm, vias 0 -> 3
- net SENSOR_2: track 0.00 -> 55.5 mm, vias 0 -> 3
- net SENSOR_3: track 0.00 -> 49.3 mm, vias 0 -> 3
- net SENSOR_5: track 0.00 -> 49.2 mm, vias 0 -> 3
- net SENSOR_6: track 0.00 -> 46.0 mm, vias 0 -> 3
- net SENSOR_24: track 0.00 -> 44.3 mm, vias 0 -> 1
- net SENSOR_4: track 0.00 -> 43.2 mm, vias 0 -> 3
- net SENSOR_23: track 0.00 -> 40.1 mm, vias 0 -> 1
- net SENSOR_22: track 0.00 -> 35.9 mm, vias 0 -> 1
- net GND: track 12.4 -> 46.7 mm, vias 4 -> 22
- net SENSOR_9: track 0.00 -> 32.9 mm, vias 0 -> 3
- net SENSOR_20: track 0.00 -> 32.5 mm, vias 0 -> 1
- net SENSOR_21: track 0.00 -> 31.7 mm, vias 0 -> 1
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- added copper zone on layer 2, net VDD
Other:
- board text added: "VAR1A REV 3.0 2019-10-05"
- board text removed: "VAR1A REV 2.0 2019-03-03"
