File: hardware/line-sensor/var1a/line-sensor-var1a-r3.brd (EAGLE design)
At the start: 112 x 60 mm, 107 parts, among them IC1 GP2S60, IC10 GP2S60, IC11 GP2S60, IC12 GP2S60, IC13 GP2S60, IC14 GP2S60, IC15 GP2S60, IC16 GP2S60, IC17 GP2S60, IC18 GP2S60, IC19 GP2S60, IC2 GP2S60, IC20 GP2S60, IC21 GP2S60, IC22 GP2S60, IC23 GP2S60, IC24 GP2S60, IC25 GP2S60, IC26 GP2S60, IC27 GP2S60, IC28 STM32L151VE, IC3 GP2S60, IC32 LM5165YDRCR, IC4 GP2S60, IC5 GP2S60, IC6 GP2S60, IC7 GP2S60, IC8 GP2S60, IC9 GP2S60, J1 MOLEX-502382-06XX, J2 MOLEX-53261-0771, J3 MOLEX-502382-03XX, Y1 CRYSTALKYOCERA-CX3225GB24000D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, Y2 CRYSTALNDK-NX3215SA

Commit message: - watchdog will now reset if either ADC or SPI didn't report in
Parts:
- removed C10, C11: 2.7p, passives:CAPACITOR-0402
- removed Y2: CRYSTALNDK-NX3215SA, passives:NDK-NX3215SA
- moved C9 5.34 mm to (70.5, 44.8), turned to 0 degrees
- moved C6 4.85 mm to (76.0, 45.0), flipped to the top, turned to 270 degrees
- moved C8 4.30 mm to (68.2, 49.2), turned to 0 degrees
- moved Y1 1.58 mm to (70.0, 47.0), turned to 180 degrees
- moved C5 0.31 mm to (72.2, 44.4)
Connections:
- removed net N$36: C10.P$1, IC28.9, Y2.1
- removed net N$37: C11.P$1, IC28.8, Y2.2
- net GND: no longer C10.P$2, C11.P$2
Routing:
- net N$33: track 9.55 -> 0.00 mm
- net N$37: track 9.18 -> 0.00 mm
- net N$36: track 7.91 -> 0.00 mm
- net N$34: track 7.43 -> 0.00 mm
- net GND: track 46.7 -> 43.0 mm, vias 22 -> 17
- net !RST: track 27.3 -> 25.9 mm, vias 0 -> 1
- net VDD: track 147.9 -> 146.8 mm, vias 38 -> 37

Commit message: - removed 32.7 kHz crystal - replaced 24 MHz crystal with 8 MHz one - fixed ring around crustal - removed all but ground layers underneath crystal location
Parts:
- C8, C9: device passives:CAPACITOR-0402 -> passives:CAPACITOR-0603
- Y1: value CRYSTALKYOCERA-CX3225GB24000D0HEQ -> CRYSTALKYOCERA-CX5032GA; device passives:KYOCERA-CX3225GB24000D0HEQ -> passives:KYOCERA-CX5032GA
- moved C8 7.77 mm to (67.8, 41.5), turned to 180 degrees
- moved C9 5.26 mm to (68.2, 49.5)
- moved Y1 2.50 mm to (68.0, 45.5), turned to 90 degrees
- moved C5 0.06 mm to (72.2, 44.4)
Connections:
- net GND: now also C8.2, C9.2; no longer C8.P$2, C9.P$2
- net N$33: now also C8.1, Y1.P$1; no longer C8.P$1, Y1.1
- net N$34: now also C9.1, Y1.P$2; no longer C9.P$1, Y1.2
Routing:
- net N$33: track 0.00 -> 10.0 mm
- net N$34: track 0.00 -> 9.23 mm
- net GND: track 43.0 -> 47.8 mm, vias 17 -> 29
- net VDD: track 146.8 -> 147.7 mm, vias 37 -> 38
