File: hardware/line-sensor/var1a/line-sensor-var1a-r3-2019-10-06.brd (EAGLE design)
At the start: 112 x 60 mm, 107 parts, among them IC1 GP2S60, IC10 GP2S60, IC11 GP2S60, IC12 GP2S60, IC13 GP2S60, IC14 GP2S60, IC15 GP2S60, IC16 GP2S60, IC17 GP2S60, IC18 GP2S60, IC19 GP2S60, IC2 GP2S60, IC20 GP2S60, IC21 GP2S60, IC22 GP2S60, IC23 GP2S60, IC24 GP2S60, IC25 GP2S60, IC26 GP2S60, IC27 GP2S60, IC28 STM32L151VE, IC3 GP2S60, IC32 LM5165YDRCR, IC4 GP2S60, IC5 GP2S60, IC6 GP2S60, IC7 GP2S60, IC8 GP2S60, IC9 GP2S60, J1 MOLEX-502382-06XX, J2 MOLEX-53261-0771, J3 MOLEX-502382-03XX, Y1 CRYSTALKYOCERA-CX3225GB24000D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, Y2 CRYSTALNDK-NX3215SA

Commit message: - fixed crystal capacitors - fixed spi2 gpio config - disabled external crystals as capacitors seems to be wrong
Parts:
- C10, C11: value 2.7p -> 2p
- C8, C9: value 4.3p -> 6p
Changed lines of the file:
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@@
 <attribute name="NAME" x="68.5" y="46.5" size="0.6" layer="22" rot="MR0" align="center"/>
 </element>
-<element name="C8" library="passives" library_urn="urn:adsk.eagle:library:9287022" package="CAPACITOR-0402" package3d_urn="urn:adsk.eagle:package:11874712/3" value="4.3p" x="65.75" y="45.75" smashed="yes" rot="MR90">
+<element name="C8" library="passives" library_urn="urn:adsk.eagle:library:9287022" package="CAPACITOR-0402" package3d_urn="urn:adsk.eagle:package:11874712/3" value="6p" x="65.75" y="45.75" smashed="yes" rot="MR90">
 <attribute name="NAME" x="65.739" y="45.75" size="0.5" layer="26" rot="MR180" align="center"/>
 </element>
-<element name="C9" library="passives" library_urn="urn:adsk.eagle:library:9287022" package="CAPACITOR-0402" package3d_urn="urn:adsk.eagle:package:11874712/3" value="4.3p" x="69.5" y="50" smashed="yes" rot="MR90">
+<element name="C9" library="passives" library_urn="urn:adsk.eagle:library:9287022" package="CAPACITOR-0402" package3d_urn="urn:adsk.eagle:package:11874712/3" value="6p" x="69.5" y="50" smashed="yes" rot="MR90">
 <attribute name="NAME" x="69.489" y="50" size="0.5" layer="26" rot="MR180" align="center"/>
 </element>
@@
 <attribute name="NAME" x="69" y="41.25" size="0.7" layer="22" rot="MR0" align="center"/>
 </element>
-<element name="C10" library="passives" library_urn="urn:adsk.eagle:library:9287022" package="CAPACITOR-0402" package3d_urn="urn:adsk.eagle:package:11874712/3" value="2.7p" x="66.5" y="42.5" smashed="yes" rot="MR0">
+<element name="C10" library="passives" library_urn="urn:adsk.eagle:library:9287022" package="CAPACITOR-0402" package3d_urn="urn:adsk.eagle:package:11874712/3" value="2p" x="66.5" y="42.5" smashed="yes" rot="MR0">
 <attribute name="NAME" x="66.5" y="42.489" size="0.5" layer="26" rot="MR90" align="center"/>
 </element>
-<element name="C11" library="passives" library_urn="urn:adsk.eagle:library:9287022" package="CAPACITOR-0402" package3d_urn="urn:adsk.eagle:package:11874712/3" value="2.7p" x="66.5" y="40" smashed="yes" rot="MR0">
+<element name="C11" library="passives" library_urn="urn:adsk.eagle:library:9287022" package="CAPACITOR-0402" package3d_urn="urn:adsk.eagle:package:11874712/3" value="2p" x="66.5" y="40" smashed="yes" rot="MR0">
 <attribute name="NAME" x="66.5" y="39.989" size="0.5" layer="26" rot="MR90" align="center"/>
+<attribute name="SPICEPREFIX" value="C" x="66.5" y="40" size="1.778" layer="28" rot="MR0" display="off"/>
 </element>
 <element name="C12" library="passives" library_urn="urn:adsk.eagle:library:9287022" package="CAPACITOR-0603" package3d_urn="urn:adsk.eagle:package:704999/4" value="1u 16V X7R" x="67" y="22.5" smashed="yes" rot="MR180">
