File: hardware/line-sensor/var1a/line-sensor-var1a-r3-2019-10-06.sch (EAGLE design)
At the start: 142 parts, among them IC1 GP2S60, IC10 GP2S60, IC11 GP2S60, IC12 GP2S60, IC13 GP2S60, IC14 GP2S60, IC15 GP2S60, IC16 GP2S60, IC17 GP2S60, IC18 GP2S60, IC19 GP2S60, IC2 GP2S60, IC20 GP2S60, IC21 GP2S60, IC22 GP2S60, IC23 GP2S60, IC24 GP2S60, IC25 GP2S60, IC26 GP2S60, IC27 GP2S60, IC28 STM32L151VE, IC3 GP2S60, IC32 LM5165YDRCR, IC4 GP2S60, IC5 GP2S60, IC6 GP2S60, IC7 GP2S60, IC8 GP2S60, IC9 GP2S60, J1 MOLEX-502382-06XX, J2 MOLEX-53261-0771, J3 MOLEX-502382-03XX, Y1 CRYSTALKYOCERA-CX3225GB24000D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, Y2 CRYSTALNDK-NX3215SA

Commit message: - fixed crystal capacitors - fixed spi2 gpio config - disabled external crystals as capacitors seems to be wrong
Parts:
- C10: value 2.7p -> 2p
- C11: value 2.7p -> 2p; SPICEPREFIX (none) -> C
- C8, C9: value 4.3p -> 6p
Changed lines of the file:
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@@
 <part name="FRAME5" library="frames" library_urn="urn:adsk.eagle:library:229" deviceset="A4L-LOC" device=""/>
 <part name="Y1" library="passives" library_urn="urn:adsk.eagle:library:9287022" deviceset="CRYSTAL" device="KYOCERA-CX3225GB24000D0HEQ" package3d_urn="urn:adsk.eagle:package:9990572/4"/>
-<part name="C8" library="passives" library_urn="urn:adsk.eagle:library:9287022" deviceset="CAPACITOR" device="0402" package3d_urn="urn:adsk.eagle:package:11874712/3" value="4.3p"/>
-<part name="C9" library="passives" library_urn="urn:adsk.eagle:library:9287022" deviceset="CAPACITOR" device="0402" package3d_urn="urn:adsk.eagle:package:11874712/3" value="4.3p"/>
+<part name="C8" library="passives" library_urn="urn:adsk.eagle:library:9287022" deviceset="CAPACITOR" device="0402" package3d_urn="urn:adsk.eagle:package:11874712/3" value="6p"/>
+<part name="C9" library="passives" library_urn="urn:adsk.eagle:library:9287022" deviceset="CAPACITOR" device="0402" package3d_urn="urn:adsk.eagle:package:11874712/3" value="6p"/>
 <part name="DGND15" library="voltage-ground" library_urn="urn:adsk.eagle:library:704746" deviceset="DGND" device=""/>
 <part name="Y2" library="passives" library_urn="urn:adsk.eagle:library:9287022" deviceset="CRYSTAL" device="NDK-NX3215SA" package3d_urn="urn:adsk.eagle:package:11610117/4"/>
-<part name="C10" library="passives" library_urn="urn:adsk.eagle:library:9287022" deviceset="CAPACITOR" device="0402" package3d_urn="urn:adsk.eagle:package:11874712/3" value="2.7p"/>
-<part name="C11" library="passives" library_urn="urn:adsk.eagle:library:9287022" deviceset="CAPACITOR" device="0402" package3d_urn="urn:adsk.eagle:package:11874712/3" value="2.7p"/>
+<part name="C10" library="passives" library_urn="urn:adsk.eagle:library:9287022" deviceset="CAPACITOR" device="0402" package3d_urn="urn:adsk.eagle:package:11874712/3" value="2p"/>
+<part name="C11" library="passives" library_urn="urn:adsk.eagle:library:9287022" deviceset="CAPACITOR" device="0402" package3d_urn="urn:adsk.eagle:package:11874712/3" value="2p">
+<attribute name="SPICEPREFIX" value="C"/>
+</part>
 <part name="DGND16" library="voltage-ground" library_urn="urn:adsk.eagle:library:704746" deviceset="DGND" device=""/>
 <part name="C12" library="passives" library_urn="urn:adsk.eagle:library:9287022" deviceset="CAPACITOR" device="0603" package3d_urn="urn:adsk.eagle:package:704999/4" value="1u 16V X7R"/>
